File: stony_skunk.sch (KiCad schematic (older format))
At the start: 33 parts, among them P1 DC/BUTTONS/CURRENT, P2 LCD, P3 RELAY, P4 NFC, P5 FTDI, P6 RESET, P7 PROG, Q1 Q_NMOS_GSD, Q2 Q_NMOS_GSD, U1 NCP1117ST33T3G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

Commit message: Clarified adjustable/optional resistors on schematic
Other:
- note added: "R3 and R4 should be adjusted to match the \ncurrent sensor, or left unpopulated for \nsensors with a built-in resistor."
Changed lines of the file:
@@
 Wire Wire Line
 	3050 4500 3050 4850
+Text Notes 4300 2600 0    39   ~ 0
+R3 and R4 should be adjusted to match the \ncurrent sensor, or left unpopulated for \nsensors with a built-in resistor.
 $EndSCHEMATC

Commit message: Replace ESP12E with Wemos D1 Mini
Parts:
- removed C1, C2: 10uF, Capacitors_SMD:C_0805, symbol C
- removed C4: 0.1uF, Capacitors_SMD:C_0603, symbol C
- removed P5: FTDI, Pin_Headers:Pin_Header_Straight_1x06, symbol CONN_01X06
- removed P6: RESET, Pin_Headers:Pin_Header_Straight_1x02, symbol CONN_01X02
- removed R10, R11, R12, R13, R14: 10K, Resistors_SMD:R_0603, symbol R
- removed U1: NCP1117ST33T3G, TO_SOT_Packages_SMD:SOT-223, symbol NCP1117ST33T3G-RESCUE-stony_skunk
- removed U3: ESP-12, timhawes:ESP-12, symbol ESP-12
- added U1: WEMOS_D1_MINI, timhawes:WEMOS_D1_MINI, symbol WEMOS_D1_MINI
Connections:
- net +3V3: now also U1.8 (3V3)
- net +5V: now also U1.9 (5V)
- net ADC: now also U1.2 (A0)
- net BUTTON_A: now also U1.13 (GPIO4/D2)
- net BUTTON_B: now also U1.14 (GPIO5/D1)
- net BUZZER: now also U1.7 (D8/GPIO15)
- net GND: now also U1.10 (GND)
- net GPIO0: now also U1.12 (GPIO0/D3)
- net PN532_RESET: now also U1.11 (GPIO2/D4)
- net RELAY: now also U1.4 (D5/GPIO14)
- net SCL: now also U1.5 (D6/GPIO12)
- net SDA: now also U1.6 (D7/GPIO13)
- no-connect marks 3 -> 4
Other:
- moved on the sheet: P7, Q2, R2, R8, R9, SP1

Commit message: Convert to Kicad v5 and fix mismatched reference in schematic (R2->R13)
Parts:
- C3: symbol C -> Device:C
- D1, D2: symbol D -> Device:D
- P1: symbol CONN_01X08 -> Connector:Screw_Terminal_01x08
- P2: symbol CONN_01X04 -> Connector:Conn_01x04_Male
- P3: symbol CONN_01X02 -> Connector:Screw_Terminal_01x02
- P4: symbol CONN_01X05 -> Connector:Conn_01x05_Male
- P7: symbol CONN_01X02 -> Connector:Conn_01x02_Male
- Q1, Q2: symbol Q_NMOS_GSD -> Device:Q_NMOS_GSD
- R1, R5, R7, R8, R9: symbol R -> Device:R
- R13: renamed from R2; symbol R -> Device:R
- R3, R4: value 22R -> 200R; symbol R -> Device:R
- R6: value 56K -> 10K; symbol R -> Device:R
- SP1: symbol SPEAKER -> Device:Speaker
- U1: symbol WEMOS_D1_MINI -> timhawes:WEMOS_D1_MINI
- U2: symbol TE_OJ_RELAY -> timhawes:TE_OJ_RELAY
Connections:
- wire segments 86 -> 101
